File: light/pcb/PNCATEHO.kicad_sch (KiCad schematic)
At the start: 51 parts, among them J1 USB_C_Receptacle_USB2.0, SW11 Boot, SW12 Boot, U1 RP2040, U2 RT9013-33GB, U3 W25Q32JVSSIQ, U4 USBLC6-2SC6, Y1 12MHz

Commit message: add button
Parts:
- SW11, SW12: footprint PNCATEHO:PADS -> PNCATEHO:SW_PUSH
Changed lines of the file:
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@@
 			)
 		)
-		(property "Footprint" "PNCATEHO:PADS"
+		(property "Footprint" "PNCATEHO:SW_PUSH"
 			(at 201.93 29.21 0)
 			(effects
@@
 			)
 		)
-		(property "Footprint" "PNCATEHO:PADS"
+		(property "Footprint" "PNCATEHO:SW_PUSH"
 			(at 179.07 29.21 0)
 			(effects

Commit message: * components moved closer to each other;  * rerouted with esd protection;  * fixed usb data differential pair length;  * changed design to be like a credit card;
Parts:
- removed R8: 10k, PNCATEHO:R_0805_2012Metric_Pad1.20x1.40mm_HandSolder, symbol PNCATEHO:R
- added C17: 100nF, PNCATEHO:C_0805_2012Metric_Pad1.18x1.45mm_HandSolder, symbol PNCATEHO:C
- D1: value Red -> RED; footprint PNCATEHO:D_0805_2012Metric_Pad1.15x1.40mm_HandSolder -> PNCATEHO:LED_0805_2012Metric_Pad1.15x1.40mm_HandSolder
- D2: value Blue -> BLUE; footprint PNCATEHO:D_0805_2012Metric_Pad1.15x1.40mm_HandSolder -> PNCATEHO:LED_0805_2012Metric_Pad1.15x1.40mm_HandSolder
- SW12: value Boot -> Reset
Connections:
- net +5V: now also C17.2
- net GND: now also C17.1
- net ~{RESET}: now also SW12.2
- net RP2040_D-: now reaches R7.2, U1.46 (USB_DM)
- net RP2040_D+: now reaches R6.2, U1.47 (USB_DP)
- net USBBN renamed USBD-
- net USBD-: now also U4.4 (I/O2); no longer U4.6 (I/O1)
- net USBBP renamed USBD+
- net USBD+: now also U4.6 (I/O1); no longer U4.4 (I/O2)
- net USB_D+ renamed USB_PROTECTED_D+
- net USB_D- renamed USB_PROTECTED_D-
Other:
- note added: "Led"
- moved on the sheet: R6, R7, U1, U4
