File: light/pcb/PNCATEHO_Welcome/PNCATEHO_Welcome.kicad_sch (KiCad schematic)
At the start: 65 parts, among them J1 USB_C_Receptacle_USB2.0, J2 Conn_01x10, J3 Conn_01x10, J4 Conn_01x05, J5 Conn_01x05, SW11 Boot, SW12 Reset, U1 RP2040, U2 RT9013-33GB, U3 W25Q32JVSSIQ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

Commit message: update footpint
Parts:
- J4, J5: footprint (none) -> PNCATEHO:PinHeader_1x05_P2.54mm_Vertical
Changed lines of the file:
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@@
 			)
 		)
-		(property "Footprint" ""
+		(property "Footprint" "PNCATEHO:PinHeader_1x05_P2.54mm_Vertical"
 			(at 372.11 111.76 0)
 			(effects
@@
 			)
 		)
-		(property "Footprint" ""
+		(property "Footprint" "PNCATEHO:PinHeader_1x05_P2.54mm_Vertical"
 			(at 372.11 96.52 0)
 			(effects
